File: Kicad Files/ATECC608A.sch (KiCad schematic (older format))
At the start: 7 parts, among them J1 Conn_01x04, U1 ATECC608A-SSHDA

Commit message: Change name LED1 and netlist
Parts:
- renumbered D1 to ON
Changed lines of the file:
@@
 Sheet 1 1
 Title "ATECC608A"
-Date "2019-09-02"
+Date "2019-09-19"
 Rev "0.1"
 Comp "Electronic Cat"
 Comment1 ""
 Comment2 ""
-Comment3 ""
+Comment3 "Montserrat Figueroa"
 Comment4 "Andres Sabas"
 $EndDescr
@@
 $EndComp
 $Comp
-L Device:LED D1
+L Device:LED ON
 U 1 1 5D6EC4F7
 P 3700 3070
-F 0 "D1" H 3693 3286 50  0000 C CNN
+F 0 "ON" H 3693 3286 50  0000 C CNN
 F 1 "LED" H 3693 3195 50  0000 C CNN
 F 2 "LED_SMD:LED_0805_2012Metric_Pad1.15x1.40mm_HandSolder" H 3700 3070 50  0001 C CNN
@@
 U 1 1 5D6EC7EA
 P 5850 2530
-F 0 "R3" H 5710 2600 50  0000 L CNN
+F 0 "R3" H 5700 2660 50  0000 L CNN
 F 1 "4K7" H 5660 2540 50  0000 L CNN
 F 2 "Resistor_SMD:R_0805_2012Metric_Pad1.15x1.40mm_HandSolder" H 5850 2530 50  0001 C CNN
@@
 U 1 1 5D6EDC5B
 P 5940 2510
-F 0 "R2" H 5999 2556 50  0000 L CNN
-F 1 "4K7" H 5999 2465 50  0000 L CNN
+F 0 "R2" H 6000 2620 50  0000 L CNN
+F 1 "4K7" H 6050 2470 50  0000 L CNN
 F 2 "Resistor_SMD:R_0805_2012Metric_Pad1.15x1.40mm_HandSolder" H 5940 2510 50  0001 C CNN
 F 3 "~" H 5940 2510 50  0001 C CNN

Commit message: Desing rules and  contour pcb
Parts:
- C1: manf# (none) -> 885012207072
- ON: manf# (none) -> 150080RS75000
- R1: manf# (none) -> RMCF0805JT180R
Changed lines of the file:
@@
 F 2 "Capacitor_SMD:C_0805_2012Metric_Pad1.15x1.40mm_HandSolder" H 6910 3050 50  0001 C CNN
 F 3 "~" H 6910 3050 50  0001 C CNN
+F 4 "885012207072" H 6910 3050 50  0001 C CNN "manf#"
 	1    6910 3050
 	1    0    0    -1
@@
 F 1 "LED" H 3693 3195 50  0000 C CNN
 F 2 "LED_SMD:LED_0805_2012Metric_Pad1.15x1.40mm_HandSolder" H 3700 3070 50  0001 C CNN
-F 3 "~" H 3700 3070 50  0001 C CNN
+F 3 " 150080RS75000 Hoja de datos" H 3700 3070 50  0001 C CNN
+F 4 "150080RS75000" H 3700 3070 50  0001 C CNN "manf#"
 	1    3700 3070
 	1    0    0    -1
@@
 F 2 "Resistor_SMD:R_0805_2012Metric_Pad1.15x1.40mm_HandSolder" H 3300 3070 50  0001 C CNN
 F 3 "~" H 3300 3070 50  0001 C CNN
+F 4 "RMCF0805JT180R" H 3300 3070 50  0001 C CNN "manf#"
 	1    3300 3070
 	0    1    1    0
